File: arm_20to10.kicad_pcb (KiCad board)
At the start: 2 copper layers, 29 x 30 mm, 12 parts, among them J1 Conn_ARM_JTAG_SWD_20, J2 Conn_ARM_JTAG_SWD_10, SW1 SW_SPDT, SW2 SW_SPST, U1 TLV70033_SOT23-5

Commit message: Final details.
Other:
- board text added: "ON|OFF TRGT EXT PWRT"
- board text added: "RESET"
- board text added: "SWDIO SWCLK SWO NC nRESET"
- board text added: "VCC GND GND NC GND"
- board text removed: "ON|OFF"
Changed lines of the file:
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@@
   (general
     (thickness 1.6)
-    (drawings 7)
+    (drawings 14)
     (tracks 101)
     (zones 0)
@@
     (descr "SW PUSH SMALL http://www.ckswitches.com/media/1457/ksa_ksl.pdf")
     (tags "SW PUSH SMALL Tactile C&K")
-    (fp_text reference SW2 (at 3.81 -2.08) (layer F.SilkS)
+    (fp_text reference SW2 (at 9.25 0.25 90) (layer F.SilkS)
       (effects (font (size 1 1) (thickness 0.15)))
     )
@@
     )
   )
+  (gr_text RESET (at 176.5 144.75) (layer F.SilkS)
+    (effects (font (size 1 1) (thickness 0.2)))
+  )
+  (gr_line (start 175.5 135.5) (end 175.5 144.5) (layer B.SilkS) (width 0.15))
+  (gr_line (start 185 144.5) (end 175.5 144.5) (layer B.SilkS) (width 0.15))
+  (gr_line (start 185 144.5) (end 185 135.5) (layer B.SilkS) (width 0.15))
+  (gr_line (start 175.5 135.5) (end 185 135.5) (layer B.SilkS) (width 0.15))
+  (gr_text "VCC\nGND\nGND\nNC\nGND" (at 179 140) (layer B.SilkS)
+    (effects (font (size 1 1) (thickness 0.2)) (justify left mirror))
+  )
+  (gr_text "SWDIO\nSWCLK\nSWO\nNC\nnRESET" (at 185 140) (layer B.SilkS)
+    (effects (font (size 1 1) (thickness 0.2)) (justify left mirror))
+  )
   (gr_line (start 161 125) (end 190 125) (layer Edge.Cuts) (width 0.1))
   (gr_line (start 161 155) (end 161 125) (layer Edge.Cuts) (width 0.1))
   (gr_line (start 190 155) (end 161 155) (layer Edge.Cuts) (width 0.1))
   (gr_line (start 190 155) (end 190 125) (layer Edge.Cuts) (width 0.1))
-  (gr_text ON|OFF (at 176.25 132.25) (layer F.SilkS)
+  (gr_text "ON|OFF\nTRGT EXT PWRT" (at 176.25 132.5) (layer F.SilkS)
     (effects (font (size 1 1) (thickness 0.2)))
   )

Commit message: Progressed PCB layout.
Parts:
- J1: footprint Connector_PinSocket_2.54mm:PinSocket_2x10_P2.54mm_Horizontal -> Connector_PinSocket_2.54mm:PinSocket_2x10_P2.54mm_Vertical; moved to B.Cu
- moved R1 68.6 mm to (119.5, 146.5)
- moved R2 68.6 mm to (119.5, 133.5)
- moved D1 65.5 mm to (119.5, 151.0), turned to 90 degrees
- moved D2 65.5 mm to (119.5, 129.0)
- moved J2 56.0 mm to (130.0, 137.8)
- moved C2 55.1 mm to (124.2, 135.8), turned to 0 degrees
- moved U1 51.8 mm to (124.2, 139.2), turned to 90 degrees
- moved SW2 50.1 mm to (122.5, 149.2)
- moved SW1 49.5 mm to (129.0, 129.0)
- moved C1 48.4 mm to (124.2, 142.8), turned to 180 degrees
- moved R3 45.7 mm to (124.2, 146.2), turned to 180 degrees
- moved J1 31.0 mm to (135.0, 129.0), turned to 180 degrees
Routing:
- net /5V: track 67.5 -> 0.00 mm, vias 2 -> 0
- net /TDI: track 30.4 -> 0.00 mm
- net /VCC: track 43.1 -> 13.2 mm, vias 1 -> 0
- net /SWCLK: track 31.2 -> 3.79 mm
- net /~RESET: track 28.6 -> 6.20 mm
- net /SWO: track 27.1 -> 6.36 mm
- net /SWDIO: track 23.9 -> 4.20 mm
- net Net-(R3-Pad2): track 13.2 -> 0.00 mm
- net Net-(C2-Pad1): track 11.7 -> 0.00 mm
- net /GND: track 9.28 -> 0.00 mm, vias 3 -> 0
- net Net-(D2-Pad2): track 3.01 -> 0.00 mm
- net Net-(D1-Pad2): track 3.01 -> 0.00 mm
Other:
- board size 29 x 30 mm -> 24 x 36 mm
- board text added: "MCU RESET"
- board text added: "ON | OFF"
- board text removed: "ON|OFF TRGT EXT PWRT"
- board text removed: "RESET"
- board text removed: "SWDIO SWCLK SWO NC nRESET"
- board text removed: "VCC GND GND NC GND"

Commit message: Progressed pcb layout.
Parts:
- turned D2 to 270 degrees
Routing:
- net /5V: track 0.00 -> 36.5 mm
- net /VCC: track 13.2 -> 32.6 mm
- net Net-(R3-Pad2): track 0.00 -> 11.8 mm
- net Net-(C2-Pad1): track 0.00 -> 10.5 mm
- net /~RESET: track 6.20 -> 13.3 mm
- net /GND: track 0.00 -> 2.82 mm
- net Net-(D2-Pad2): track 0.00 -> 2.45 mm
- net Net-(D1-Pad2): track 0.00 -> 2.45 mm
Other:
- board text added: "20-pin IDC JTAG to Cortex Debug Connector"
- board text added: "Nuno Sousa 05/2020"
- board text added: "SPLY PWR TO TRGT"
Changed lines of the file:
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@@
   (general
     (thickness 1.6)
-    (drawings 12)
-    (tracks 17)
+    (drawings 19)
+    (tracks 56)
     (zones 0)
     (modules 12)
@@
   )
   (module LED_SMD:LED_0805_2012Metric_Pad1.15x1.40mm_HandSolder (layer F.Cu)
-    (at 119.5 129 90)
+    (at 119.5 129 270)
     (descr "LED SMD 0805 (2012 Metric), square (rectangular) end terminal, IPC_7351 nominal, (Body size source: https://docs.google.com/spreadsheets/d/1BsfQQcO9C6DZCsRaXUlFlo91Tg2WpOkGARC1WS5S8t0/edit?usp=sharing), generated with kicad-footprint-generator")
     (tags "LED handsolder")
     (attr smd)
-    (fp_text reference D2 (at 0 -1.65 90) (layer F.SilkS)
+    (fp_text reference D2 (at 0 1.6 90) (layer F.SilkS)
       (effects (font (size 1 1) (thickness 0.15)))
     )
@@
     (fp_line (start -0.7 -0.6) (end -1 -0.3) (layer F.Fab) (width 0.1))
     (fp_line (start 1 -0.6) (end -0.7 -0.6) (layer F.Fab) (width 0.1))
-    (pad 2 smd roundrect (at 1.025 0 90) (size 1.15 1.4) (layers F.Cu F.Paste F.Mask) (roundrect_rratio 0.217391)
+    (pad 2 smd roundrect (at 1.025 0 270) (size 1.15 1.4) (layers F.Cu F.Paste F.Mask) (roundrect_rratio 0.217391)
       (net 6 "Net-(D2-Pad2)"))
-    (pad 1 smd roundrect (at -1.025 0 90) (size 1.15 1.4) (layers F.Cu F.Paste F.Mask) (roundrect_rratio 0.217391)
+    (pad 1 smd roundrect (at -1.025 0 270) (size 1.15 1.4) (layers F.Cu F.Paste F.Mask) (roundrect_rratio 0.217391)
       (net 9 /GND))
     (model ${KISYS3DMOD}/LED_SMD.3dshapes/LED_0805_2012Metric.wrl
@@
     )
   )
+  (gr_line (start 128.5 147.5) (end 128.5 157) (layer B.SilkS) (width 0.15))
+  (gr_line (start 124.5 147.5) (end 128.5 147.5) (layer B.SilkS) (width 0.15))
+  (gr_line (start 124.5 157) (end 124.5 147.5) (layer B.SilkS) (width 0.15))
+  (gr_line (start 128.5 157) (end 124.5 157) (layer B.SilkS) (width 0.15))
+  (gr_text "Nuno Sousa\n05/2020" (at 126.5 152.3 270) (layer B.SilkS)
+    (effects (font (size 1 1) (thickness 0.2)) (justify mirror))
+  )
+  (gr_text "20-pin IDC JTAG\nto\nCortex Debug Connector" (at 122 139.5 270) (layer B.SilkS)
+    (effects (font (size 1 1) (thickness 0.2)) (justify mirror))
+  )
+  (gr_text "SPLY PWR\nTO TRGT" (at 136.2 124.8) (layer F.SilkS)
+    (effects (font (size 1 1) (thickness 0.2)))
+  )
   (gr_text "MCU RESET" (at 126.5 156.75 180) (layer F.SilkS)
     (effects (font (size 1 1) (thickness 0.2)))
@@
     (effects (font (size 1 1) (thickness 0.2) italic))
   )
+  (segment (start 123.38 139.32) (end 125.2 139.32) (width 0.5) (layer F.Cu) (net 1))
+  (segment (start 123.3 140.35) (end 123.3 139.4) (width 0.5) (layer F.Cu) (net 1))
+  (segment (start 125.2 139.32) (end 125.2 140.35) (width 0.5) (layer F.Cu) (net 1))
+  (segment (start 123.3 139.4) (end 123.38 139.32) (width 0.5) (layer F.Cu) (net 1))
+  (segment (start 125.275 140.425) (end 125.2 140.35) (width 0.5) (layer F.Cu) (net 1))
+  (segment (start 125.275 142.75) (end 125.275 140.425) (width 0.5) (layer F.Cu) (net 1))
+  (segment (start 121.175 144.5) (end 124.225 144.5) (width 0.5) (layer F.Cu) (net 1))
+  (segment (start 119.5 145.475) (end 120.2 145.475) (width 0.5) (layer F.Cu) (net 1))
+  (segment (start 125.275 143.45) (end 125.275 142.75) (width 0.5) (layer F.Cu) (net 1))
+  (segment (start 124.225 144.5) (end 125.275 143.45) (width 0.5) (layer F.Cu) (net 1))
+  (segment (start 120.2 145.475) (end 121.175 144.5) (width 0.5) (layer F.Cu) (net 1))
+  (segment (start 120.9 150.2) (end 120.9 146.2) (width 0.5) (layer F.Cu) (net 1))
+  (segment (start 122.6 144.5) (end 124.225 144.5) (width 0.5) (layer F.Cu) (net 1))
+  (segment (start 135 151.86) (end 122.56 151.86) (width 0.5) (layer F.Cu) (net 1))
+  (segment (start 120.9 146.2) (end 122.6 144.5) (width 0.5) (layer F.Cu) (net 1))
+  (segment (start 122.56 151.86) (end 120.9 150.2) (width 0.5) (layer F.Cu) (net 1))
   (segment (start 124 129) (end 125.7 127.3) (width 0.5) (layer F.Cu) (net 3))
   (segment (start 135 127.65) (end 135 129) (width 0.5) (layer F.Cu) (net 3))
   (segment (start 134.65 127.3) (end 135 127.65) (width 0.5) (layer F.Cu) (net 3))
   (segment (start 125.7 127.3) (end 134.65 127.3) (width 0.5) (layer F.Cu) (net 3))
-  (segment (start 131.27 143.537106) (end 131.27 142.83) (width 0.5) (layer F.Cu) (net 10))
+  (segment (start 133.65 129) (end 135 129) (width 0.5) (layer F.Cu) (net 3))
+  (segment (start 130 132.65) (end 133.65 129) (width 0.5) (layer F.Cu) (net 3))
+  (segment (start 130 137.75) (end 130 132.65) (width 0.5) (layer F.Cu) (net 3))
+  (segment (start 124 130.725) (end 124 129.989949) (width 0.5) (layer F.Cu) (net 3))
+  (segment (start 124 129.989949) (end 124 129) (width 0.5) (layer F.Cu) (net 3))
+  (segment (start 120.2 134.525) (end 124 130.725) (width 0.5) (layer F.Cu) (net 3))
+  (segment (start 119.5 134.525) (end 120.2 134.525) (width 0.5) (layer F.Cu) (net 3))
+  (segment (start 123.3 135.825) (end 123.225 135.75) (width 0.5) (layer F.Cu) (net 4))
+  (segment (start 123.3 138.15) (end 123.3 135.825) (width 0.5) (layer F.Cu) (net 4))
+  (segment (start 126.5 129) (end 126.5 130.8) (width 0.5) (layer F.Cu) (net 4))
+  (segment (start 123.225 134.075) (end 123.225 135.75) (width 0.5) (layer F.Cu) (net 4))
+  (segment (start 126.5 130.8) (end 123.225 134.075) (width 0.5) (layer F.Cu) (net 4))
+  (segment (start 119.5 149.975) (end 119.5 147.525) (width 0.5) (layer F.Cu) (net 5))
+  (segment (start 119.5 132.475) (end 119.5 130.025) (width 0.5) (layer F.Cu) (net 6))
+  (segment (start 124.25 141.725) (end 124.25 140.35) (width 0.5) (layer F.Cu) (net 9))
+  (segment (start 123.225 142.75) (end 124.25 141.725) (width 0.5) (layer F.Cu) (net 9))
   (segment (start 131.27 144.252081) (end 131.27 143.537106) (width 0.5) (layer F.Cu) (net 10))
   (segment (start 133.797919 146.78) (end 131.27 144.252081) (width 0.5) (layer F.Cu) (net 10))
   (segment (start 135 146.78) (end 133.797919 146.78) (width 0.5) (layer F.Cu) (net 10))
+  (segment (start 131.27 143.537106) (end 131.27 142.83) (width 0.5) (layer F.Cu) (net 10))
+  (segment (start 128.557106 146.25) (end 131.27 143.537106) (width 0.5) (layer F.Cu) (net 10))
+  (segment (start 125.275 146.25) (end 128.557106 146.25) (width 0.5) (layer F.Cu) (net 10))
   (segment (start 132.9 141.2) (end 131.99 140.29) (width 0.5) (layer F.Cu) (net 11))
   (segment (start 132.9 142.9) (end 132.9 141.2) (width 0.5) (layer F.Cu) (net 11))
@@
   (segment (start 132.4 136.62) (end 131.27 137.75) (width 0.5) (layer F.Cu) (net 14))
   (segment (start 135 136.62) (end 132.4 136.62) (width 0.5) (layer F.Cu) (net 14))
+  (segment (start 123.225 148.525) (end 122.5 149.25) (width 0.5) (layer F.Cu) (net 18))
+  (segment (start 123.225 146.25) (end 123.225 148.525) (width 0.5) (layer F.Cu) (net 18))
+  (segment (start 123.225 146.95) (end 123.225 146.25) (width 0.5) (layer F.Cu) (net 18))
+  (segment (start 125.525 149.25) (end 123.225 146.95) (width 0.5) (layer F.Cu) (net 18))
+  (segment (start 130.12 149.25) (end 125.525 149.25) (width 0.5) (layer F.Cu) (net 18))
   (zone (net 9) (net_name /GND) (layer F.Cu) (hatch edge 0.508)
     (connect_pads (clearance 0.25))

Commit message: Final updates.
Routing:
- net /TDI: track 0.00 -> 19.9 mm
- net /GND: vias 0 -> 6
Changed lines of the file:
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@@
     (thickness 1.6)
     (drawings 19)
-    (tracks 56)
+    (tracks 72)
     (zones 0)
     (modules 12)
@@
   (segment (start 120.9 146.2) (end 122.6 144.5) (width 0.5) (layer F.Cu) (net 1))
   (segment (start 122.56 151.86) (end 120.9 150.2) (width 0.5) (layer F.Cu) (net 1))
+  (segment (start 133.797919 134.08) (end 135 134.08) (width 0.5) (layer B.Cu) (net 2))
+  (segment (start 128.999999 143.310001) (end 128.999999 136.849999) (width 0.5) (layer B.Cu) (net 2))
+  (segment (start 131.769998 134.08) (end 133.797919 134.08) (width 0.5) (layer B.Cu) (net 2))
+  (segment (start 129.519999 143.830001) (end 128.999999 143.310001) (width 0.5) (layer B.Cu) (net 2))
+  (segment (start 128.999999 136.849999) (end 131.769998 134.08) (width 0.5) (layer B.Cu) (net 2))
+  (segment (start 132.270001 143.310001) (end 131.750001 143.830001) (width 0.5) (layer B.Cu) (net 2))
+  (segment (start 131.750001 143.830001) (end 129.519999 143.830001) (width 0.5) (layer B.Cu) (net 2))
+  (segment (start 132.270001 141.852895) (end 132.270001 143.310001) (width 0.5) (layer B.Cu) (net 2))
+  (segment (start 131.977106 141.56) (end 132.270001 141.852895) (width 0.5) (layer B.Cu) (net 2))
+  (segment (start 131.27 141.56) (end 131.977106 141.56) (width 0.5) (layer B.Cu) (net 2))
   (segment (start 124 129) (end 125.7 127.3) (width 0.5) (layer F.Cu) (net 3))
   (segment (start 135 127.65) (end 135 129) (width 0.5) (layer F.Cu) (net 3))
@@
   (segment (start 124.25 141.725) (end 124.25 140.35) (width 0.5) (layer F.Cu) (net 9))
   (segment (start 123.225 142.75) (end 124.25 141.725) (width 0.5) (layer F.Cu) (net 9))
+  (via (at 127 134.5) (size 1) (drill 0.5) (layers F.Cu B.Cu) (net 9))
+  (via (at 127 137) (size 1) (drill 0.5) (layers F.Cu B.Cu) (net 9))
+  (via (at 127 141.5) (size 1) (drill 0.5) (layers F.Cu B.Cu) (net 9))
+  (via (at 127 144) (size 1) (drill 0.5) (layers F.Cu B.Cu) (net 9))
+  (via (at 123.5 150.86) (size 1) (drill 0.5) (layers F.Cu B.Cu) (net 9))
+  (via (at 131 146) (size 1) (drill 0.5) (layers F.Cu B.Cu) (net 9))
   (segment (start 131.27 144.252081) (end 131.27 143.537106) (width 0.5) (layer F.Cu) (net 10))
   (segment (start 133.797919 146.78) (end 131.27 144.252081) (width 0.5) (layer F.Cu) (net 10))
@@
   (segment (start 128.557106 146.25) (end 131.27 143.537106) (width 0.5) (layer F.Cu) (net 10))
   (segment (start 125.275 146.25) (end 128.557106 146.25) (width 0.5) (layer F.Cu) (net 10))
-  (segment (start 132.9 141.2) (end 131.99 140.29) (width 0.5) (layer F.Cu) (net 11))
-  (segment (start 132.9 142.9) (end 132.9 141.2) (width 0.5) (layer F.Cu) (net 11))
-  (segment (start 131.99 140.29) (end 131.27 140.29) (width 0.5) (layer F.Cu) (net 11))
+  (segment (start 133.3 141.4) (end 132.19 140.29) (width 0.5) (layer F.Cu) (net 11))
+  (segment (start 133.3 143.3) (end 133.3 141.4) (width 0.5) (layer F.Cu) (net 11))
+  (segment (start 132.19 140.29) (end 131.27 140.29) (width 0.5) (layer F.Cu) (net 11))
   (segment (start 135 144.24) (end 134.24 144.24) (width 0.5) (layer F.Cu) (net 11))
-  (segment (start 134.24 144.24) (end 132.9 142.9) (width 0.5) (layer F.Cu) (net 11))
+  (segment (start 134.24 144.24) (end 133.3 143.3) (width 0.5) (layer F.Cu) (net 11))
   (segment (start 134.86 139.02) (end 135 139.16) (width 0.5) (layer F.Cu) (net 13))
   (segment (start 131.27 139.02) (end 134.86 139.02) (width 0.5) (layer F.Cu) (net 13))
