File: arm_20to10.sch (KiCad schematic (older format))
At the start: 12 parts, among them J1 Conn_ARM_JTAG_SWD_20, J2 Conn_ARM_JTAG_SWD_10, SW1 SW_SPDT, SW2 SW_SPST, U1 TLV70033_SOT23-5

Commit message: Progressed PCB layout.
Parts:
- J1: footprint Connector_PinSocket_2.54mm:PinSocket_2x10_P2.54mm_Horizontal -> Connector_PinSocket_2.54mm:PinSocket_2x10_P2.54mm_Vertical
Changed lines of the file:
@@
 F 0 "J1" H 3371 4896 50  0000 R CNN
 F 1 "Conn_ARM_JTAG_SWD_20" H 3371 4805 50  0000 R CNN
-F 2 "Connector_PinSocket_2.54mm:PinSocket_2x10_P2.54mm_Horizontal" H 4350 3800 50  0001 L TNN
+F 2 "Connector_PinSocket_2.54mm:PinSocket_2x10_P2.54mm_Vertical" H 4350 3800 50  0001 L TNN
 F 3 "http://infocenter.arm.com/help/topic/com.arm.doc.dui0499b/DUI0499B_system_design_reference.pdf" V 3550 3600 50  0001 C CNN
 F 4 "SFH11-PBPC-D10-RA-BK" H 3900 4850 50  0001 C CNN "Manufacturer Part Number"

Commit message: Final updates.
Parts:
- J1: Manufacturer Part Number SFH11-PBPC-D10-RA-BK -> SFH11-PBPC-D10-ST-BK
- R3: Manufacturer Part Number (none) -> CR0805-JW-331ELF
Changed lines of the file:
@@
 F 2 "Connector_PinSocket_2.54mm:PinSocket_2x10_P2.54mm_Vertical" H 4350 3800 50  0001 L TNN
 F 3 "http://infocenter.arm.com/help/topic/com.arm.doc.dui0499b/DUI0499B_system_design_reference.pdf" V 3550 3600 50  0001 C CNN
-F 4 "SFH11-PBPC-D10-RA-BK" H 3900 4850 50  0001 C CNN "Manufacturer Part Number"
+F 4 "SFH11-PBPC-D10-ST-BK" H 3900 4850 50  0001 C CNN "Manufacturer Part Number"
 	1    3900 4850
 	1    0    0    -1
@@
 F 2 "Resistor_SMD:R_0805_2012Metric_Pad1.15x1.40mm_HandSolder" V 9130 3000 50  0001 C CNN
 F 3 "~" H 9200 3000 50  0001 C CNN
+F 4 "CR0805-JW-331ELF" H 9200 3000 50  0001 C CNN "Manufacturer Part Number"
 	1    9200 3000
 	1    0    0    -1

Commit message: Update arm_20to10.sch
Parts:
- C1, C2: Manufacturer Part Number (none) -> CC0805MKX7R7BB105
- D1, D2: Manufacturer Part Number (none) -> 5988120107F
- R1, R2: value R -> 330R; Manufacturer Part Number (none) -> CR0805-JW-331ELF
Changed lines of the file:
@@
 F 2 "Capacitor_SMD:C_0805_2012Metric_Pad1.15x1.40mm_HandSolder" H 4238 1900 50  0001 C CNN
 F 3 "~" H 4200 2050 50  0001 C CNN
+F 4 "CC0805MKX7R7BB105" H 4200 2050 50  0001 C CNN "Manufacturer Part Number"
 	1    4200 2050
 	1    0    0    -1
@@
 F 2 "Capacitor_SMD:C_0805_2012Metric_Pad1.15x1.40mm_HandSolder" H 5788 1900 50  0001 C CNN
 F 3 "~" H 5750 2050 50  0001 C CNN
+F 4 "CC0805MKX7R7BB105" H 5750 2050 50  0001 C CNN "Manufacturer Part Number"
 	1    5750 2050
 	1    0    0    -1
@@
 P 3500 2050
 F 0 "R1" H 3570 2096 50  0000 L CNN
-F 1 "R" H 3570 2005 50  0000 L CNN
+F 1 "330R" H 3570 2005 50  0000 L CNN
 F 2 "Resistor_SMD:R_0805_2012Metric_Pad1.15x1.40mm_HandSolder" V 3430 2050 50  0001 C CNN
 F 3 "~" H 3500 2050 50  0001 C CNN
+F 4 "CR0805-JW-331ELF" H 3500 2050 50  0001 C CNN "Manufacturer Part Number"
 	1    3500 2050
 	1    0    0    -1
@@
 P 7000 2150
 F 0 "R2" H 7070 2196 50  0000 L CNN
-F 1 "R" H 7070 2105 50  0000 L CNN
+F 1 "330R" H 7070 2105 50  0000 L CNN
 F 2 "Resistor_SMD:R_0805_2012Metric_Pad1.15x1.40mm_HandSolder" V 6930 2150 50  0001 C CNN
 F 3 "~" H 7000 2150 50  0001 C CNN
+F 4 "CR0805-JW-331ELF" H 7000 2150 50  0001 C CNN "Manufacturer Part Number"
 	1    7000 2150
 	1    0    0    -1
@@
 F 1 "LED" V 3448 2283 50  0000 R CNN
 F 2 "LED_SMD:LED_0805_2012Metric_Pad1.15x1.40mm_HandSolder" H 3500 2400 50  0001 C CNN
-F 3 "~" H 3500 2400 50  0001 C CNN
+F 3 "https://media.digikey.com/pdf/Data%20Sheets/Dialight%20PDFs/598_Series_0805_Pkg.pdf" H 3500 2400 50  0001 C CNN
+F 4 "5988120107F" H 3500 2400 50  0001 C CNN "Manufacturer Part Number"
 	1    3500 2400
 	0    -1   -1   0
@@
 F 1 "LED" V 6948 2383 50  0000 R CNN
 F 2 "LED_SMD:LED_0805_2012Metric_Pad1.15x1.40mm_HandSolder" H 7000 2500 50  0001 C CNN
-F 3 "~" H 7000 2500 50  0001 C CNN
+F 3 "https://media.digikey.com/pdf/Data%20Sheets/Dialight%20PDFs/598_Series_0805_Pkg.pdf" H 7000 2500 50  0001 C CNN
+F 4 "5988120107F" H 7000 2500 50  0001 C CNN "Manufacturer Part Number"
 	1    7000 2500
 	0    -1   -1   0
